Commit message: feat(urdf): render Unitree G1 + Go2 from official URDFs with real meshes
Replaces the hand-authored primitive-only G1 and Go2 URDFs with the
upstream unitreerobotics descriptors and a JS-side mesh loader that
fetches, parses (STL / Collada / glTF via three.js), and inlines triangle
data into the document before the editor sees it.

Also includes:
- URDF primitive centering fix: Cube/Cylinder are now wrapped in a
  Translate that puts their geometry on the link frame origin (URDF
  semantics) instead of leaving them anchored at the kernel's default
  corner / XY-plane.
- Eval handles ImportedMesh in the assembly part-def path (was returning
  None, silently dropping every URDF mesh visual).
- CRDT migration handles MeshImport so URDF drag-drops without a mesh
  manifest still round-trip through the migration.
- Camera auto-fit considers instance FK transforms (assembly mode used
  to fit on link-local geometry collapsed at the origin).
- Physics body builder tolerates unresolvable STL paths and recognises
  inline ImportedMesh data.
- ColladaLoader's Z_UP → Y_UP scene rotation is cleared so DAE vertices
  stay in the URDF's authored Z-up frame (otherwise every leg was 90°
  off-axis from where its joint anchored it).

Co-Authored-By: Claude Opus 4.7 (1M context) <noreply@anthropic.com>

File: examples/unitree-g1.urdf (robot description, URDF)
Before this commit: robot unitree_g1, 27 links, 26 joints
Links:
- removed link left_foot_link
- removed link left_hand_link
- removed link left_wrist_roll_link
- removed link right_foot_link
- removed link right_hand_link
- removed link right_wrist_roll_link
- added link d435_link
- added link imu_in_pelvis
- added link imu_in_torso
- added link left_ankle_roll_link, mass 0.608; collision sphere radius=0.005; collision sphere radius=0.005
- added link left_wrist_roll_rubber_hand, mass 0.35692864; collision mesh filename=meshes/left_wrist_roll_rubber_hand.STL; visual mesh filename=meshes/left_wrist_roll_rubber_hand.STL
- added link logo_link, mass 0.001; collision mesh filename=meshes/logo_link.STL; visual mesh filename=meshes/logo_link.STL
- added link mid360_link
- added link pelvis_contour_link, mass 0.001; collision mesh filename=meshes/pelvis_contour_link.STL; visual mesh filename=meshes/pelvis_contour_link.STL
- added link right_ankle_roll_link, mass 0.608; collision sphere radius=0.005; collision sphere radius=0.005
- added link right_wrist_roll_rubber_hand, mass 0.35692864; collision mesh filename=meshes/right_wrist_roll_rubber_hand.STL; visual mesh filename=meshes/right_wrist_roll_rubber_hand.STL
- added link waist_support_link, mass 0.001; collision mesh filename=meshes/waist_support_link.STL; visual mesh filename=meshes/waist_support_link.STL
- added link waist_yaw_fixed_link, mass 0.244; visual mesh filename=meshes/waist_yaw_link.STL
- link head_link: mass 0.90 -> 1.036; geometry collision mesh filename=meshes/head_link.STL; visual mesh filename=meshes/head_link.STL
- link left_ankle_pitch_link: mass 0.30 -> 0.074; geometry collision mesh filename=meshes/left_ankle_pitch_link.STL; visual mesh filename=meshes/left_ankle_pitch_link.STL
- link left_elbow_link: mass 0.50 -> 0.6; geometry collision mesh filename=meshes/left_elbow_link.STL; visual mesh filename=meshes/left_elbow_link.STL
- link left_hip_pitch_link: mass 1.85 -> 1.35; geometry collision mesh filename=meshes/left_hip_pitch_link.STL; visual mesh filename=meshes/left_hip_pitch_link.STL
- link left_hip_roll_link: mass 0.80 -> 1.52; geometry collision mesh filename=meshes/left_hip_roll_link.STL; visual mesh filename=meshes/left_hip_roll_link.STL
- link left_hip_yaw_link: mass 0.80 -> 1.702; geometry collision mesh filename=meshes/left_hip_yaw_link.STL; visual mesh filename=meshes/left_hip_yaw_link.STL
- link left_knee_link: mass 1.10 -> 1.932; geometry collision mesh filename=meshes/left_knee_link.STL; visual mesh filename=meshes/left_knee_link.STL
- link left_shoulder_pitch_link: mass 0.55 -> 0.718; geometry collision cylinder length=0.05 radius=0.03; visual mesh filename=meshes/left_shoulder_pitch_link.STL
- link left_shoulder_roll_link: mass 0.55 -> 0.643; geometry collision cylinder length=0.03 radius=0.03; visual mesh filename=meshes/left_shoulder_roll_link.STL
- link left_shoulder_yaw_link: mass 0.65 -> 0.734; geometry collision mesh filename=meshes/left_shoulder_yaw_link.STL; visual mesh filename=meshes/left_shoulder_yaw_link.STL
- link pelvis: mass 3.50 -> 3.813; geometry visual mesh filename=meshes/pelvis.STL
- link right_ankle_pitch_link: mass 0.30 -> 0.074; geometry collision mesh filename=meshes/right_ankle_pitch_link.STL; visual mesh filename=meshes/right_ankle_pitch_link.STL
- link right_elbow_link: mass 0.50 -> 0.6; geometry collision mesh filename=meshes/right_elbow_link.STL; visual mesh filename=meshes/right_elbow_link.STL
- link right_hip_pitch_link: mass 1.85 -> 1.35; geometry collision mesh filename=meshes/right_hip_pitch_link.STL; visual mesh filename=meshes/right_hip_pitch_link.STL
- link right_hip_roll_link: mass 0.80 -> 1.52; geometry collision mesh filename=meshes/right_hip_roll_link.STL; visual mesh filename=meshes/right_hip_roll_link.STL
- link right_hip_yaw_link: mass 0.80 -> 1.702; geometry collision mesh filename=meshes/right_hip_yaw_link.STL; visual mesh filename=meshes/right_hip_yaw_link.STL
- link right_knee_link: mass 1.10 -> 1.932; geometry collision mesh filename=meshes/right_knee_link.STL; visual mesh filename=meshes/right_knee_link.STL
- link right_shoulder_pitch_link: mass 0.55 -> 0.718; geometry collision cylinder length=0.05 radius=0.03; visual mesh filename=meshes/right_shoulder_pitch_link.STL
- link right_shoulder_roll_link: mass 0.55 -> 0.643; geometry collision cylinder length=0.03 radius=0.03; visual mesh filename=meshes/right_shoulder_roll_link.STL
- link right_shoulder_yaw_link: mass 0.65 -> 0.734; geometry collision mesh filename=meshes/right_shoulder_yaw_link.STL; visual mesh filename=meshes/right_shoulder_yaw_link.STL
- link torso_link: mass 6.50 -> 8.562; geometry collision mesh filename=meshes/torso_link.STL; visual mesh filename=meshes/torso_link.STL
Joints:
- removed joint head_fixed_joint
- removed joint left_hand_fixed_joint
- removed joint right_hand_fixed_joint
- added joint d435_joint: type fixed, parent torso_link, child d435_link, origin xyz=0.0576235 0.01753 0.41987 rpy=0 0.8307767239493009 0
- added joint head_joint: type fixed, parent torso_link, child head_link, origin xyz=0.0039635 0 -0.054 rpy=0 0 0
- added joint imu_in_pelvis_joint: type fixed, parent pelvis, child imu_in_pelvis, origin xyz=0.04525 0 -0.08339 rpy=0 0 0
- added joint imu_in_torso_joint: type fixed, parent torso_link, child imu_in_torso, origin xyz=-0.03959 -0.00224 0.13792 rpy=0 0 0
- added joint logo_joint: type fixed, parent torso_link, child logo_link, origin xyz=0.0039635 0 -0.054 rpy=0 0 0
- added joint mid360_joint: type fixed, parent torso_link, child mid360_link, origin xyz=0.0002835 0.00003 0.40618 rpy=0 0.04014257279586953 0
- added joint pelvis_contour_joint: type fixed, parent pelvis, child pelvis_contour_link
- added joint waist_support_joint: type fixed, parent torso_link, child waist_support_link, origin xyz=0.0039635 0 -0.054 rpy=0 0 0
- added joint waist_yaw_fixed_joint: type fixed, parent torso_link, child waist_yaw_fixed_link, origin xyz=0.0039635 0 -0.054 rpy=0 0 0
- joint left_ankle_pitch_joint: limit lower=-0.87 upper=0.52 effort=35 velocity=32 -> lower=-0.87267 upper=0.5236 effort=35 velocity=30; origin xyz=0 0 -0.20 rpy=0 0 0 -> xyz=0 -9.4445E-05 -0.30001 rpy=0 0 0
- joint left_ankle_roll_joint: child left_foot_link -> left_ankle_roll_link; limit lower=-0.26 upper=0.26 effort=35 velocity=32 -> lower=-0.2618 upper=0.2618 effort=35 velocity=30; origin xyz=0 0 0 rpy=0 0 0 -> xyz=0 0 -0.017558 rpy=0 0 0
- joint left_elbow_joint: limit lower=-1.05 upper=2.27 effort=40 velocity=32 -> lower=-1.0472 upper=2.0944 effort=25 velocity=37; origin xyz=0 0 -0.17 rpy=0 0 0 -> xyz=0.015783 0 -0.080518 rpy=0 0 0
- joint left_hip_pitch_joint: limit lower=-1.75 upper=2.88 effort=139 velocity=20 -> lower=-2.5307 upper=2.8798 effort=88 velocity=32; origin xyz=0 0 0 rpy=0 0 0 -> xyz=0 0.064452 -0.1027 rpy=0 0 0; parent left_hip_roll_link -> pelvis
- joint left_hip_roll_joint: limit lower=-0.43 upper=2.53 effort=139 velocity=20 -> lower=-0.5236 upper=2.9671 effort=88 velocity=32; origin xyz=0 0 -0.04 rpy=0 0 0 -> xyz=0 0.052 -0.030465 rpy=0 -0.1749 0; parent left_hip_yaw_link -> left_hip_pitch_link
- joint left_hip_yaw_joint: limit lower=-0.43 upper=0.43 effort=88 velocity=32 -> lower=-2.7576 upper=2.7576 effort=88 velocity=32; origin xyz=0 0.07 -0.06 rpy=0 0 0 -> xyz=0.025001 0 -0.12412 rpy=0 0 0; parent pelvis -> left_hip_roll_link
- joint left_knee_joint: limit lower=-0.087 upper=2.88 effort=139 velocity=20 -> lower=-0.087267 upper=2.8798 effort=139 velocity=20; origin xyz=0 0 -0.21 rpy=0 0 0 -> xyz=-0.078273 0.0021489 -0.17734 rpy=0 0.1749 0; parent left_hip_pitch_link -> left_hip_yaw_link
- joint left_shoulder_pitch_joint: limit lower=-3.14 upper=1.57 effort=40 velocity=32 -> lower=-3.0892 upper=2.6704 effort=25 velocity=37; origin xyz=0 0.155 0.225 rpy=0 0 0 -> xyz=0.0039563 0.10022 0.23778 rpy=0.27931 5.4949E-05 -0.00019159
- joint left_shoulder_roll_joint: limit lower=-1.57 upper=2.27 effort=40 velocity=32 -> lower=-1.5882 upper=2.2515 effort=25 velocity=37; origin xyz=0 0.04 0 rpy=0 0 0 -> xyz=0 0.038 -0.013831 rpy=-0.27925 0 0
- joint left_shoulder_yaw_joint: limit lower=-2.62 upper=2.62 effort=40 velocity=32 -> lower=-2.618 upper=2.618 effort=25 velocity=37; origin xyz=0 0 0 rpy=0 0 0 -> xyz=0 0.00624 -0.1032 rpy=0 0 0
- joint left_wrist_roll_joint: axis 0 0 1 -> 1 0 0; child left_wrist_roll_link -> left_wrist_roll_rubber_hand; limit lower=-1.97 upper=1.97 effort=18 velocity=32 -> lower=-1.972222054 upper=1.972222054 effort=25 velocity=37; origin xyz=0 0 -0.18 rpy=0 0 0 -> xyz=0.100 0.00188791 -0.010 rpy=0 0 0
- joint right_ankle_pitch_joint: limit lower=-0.87 upper=0.52 effort=35 velocity=32 -> lower=-0.87267 upper=0.5236 effort=35 velocity=30; origin xyz=0 0 -0.20 rpy=0 0 0 -> xyz=0 9.4445E-05 -0.30001 rpy=0 0 0
- joint right_ankle_roll_joint: child right_foot_link -> right_ankle_roll_link; limit lower=-0.26 upper=0.26 effort=35 velocity=32 -> lower=-0.2618 upper=0.2618 effort=35 velocity=30; origin xyz=0 0 0 rpy=0 0 0 -> xyz=0 0 -0.017558 rpy=0 0 0
- joint right_elbow_joint: limit lower=-1.05 upper=2.27 effort=40 velocity=32 -> lower=-1.0472 upper=2.0944 effort=25 velocity=37; origin xyz=0 0 -0.17 rpy=0 0 0 -> xyz=0.015783 0 -0.080518 rpy=0 0 0
- joint right_hip_pitch_joint: limit lower=-1.75 upper=2.88 effort=139 velocity=20 -> lower=-2.5307 upper=2.8798 effort=88 velocity=32; origin xyz=0 0 0 rpy=0 0 0 -> xyz=0 -0.064452 -0.1027 rpy=0 0 0; parent right_hip_roll_link -> pelvis
- joint right_hip_roll_joint: limit lower=-2.53 upper=0.43 effort=139 velocity=20 -> lower=-2.9671 upper=0.5236 effort=88 velocity=32; origin xyz=0 0 -0.04 rpy=0 0 0 -> xyz=0 -0.052 -0.030465 rpy=0 -0.1749 0; parent right_hip_yaw_link -> right_hip_pitch_link
- joint right_hip_yaw_joint: limit lower=-0.43 upper=0.43 effort=88 velocity=32 -> lower=-2.7576 upper=2.7576 effort=88 velocity=32; origin xyz=0 -0.07 -0.06 rpy=0 0 0 -> xyz=0.025001 0 -0.12412 rpy=0 0 0; parent pelvis -> right_hip_roll_link
- joint right_knee_joint: limit lower=-0.087 upper=2.88 effort=139 velocity=20 -> lower=-0.087267 upper=2.8798 effort=139 velocity=20; origin xyz=0 0 -0.21 rpy=0 0 0 -> xyz=-0.078273 -0.0021489 -0.17734 rpy=0 0.1749 0; parent right_hip_pitch_link -> right_hip_yaw_link
- joint right_shoulder_pitch_joint: limit lower=-3.14 upper=1.57 effort=40 velocity=32 -> lower=-3.0892 upper=2.6704 effort=25 velocity=37; origin xyz=0 -0.155 0.225 rpy=0 0 0 -> xyz=0.0039563 -0.10021 0.23778 rpy=-0.27931 5.4949E-05 0.00019159
- joint right_shoulder_roll_joint: limit lower=-2.27 upper=1.57 effort=40 velocity=32 -> lower=-2.2515 upper=1.5882 effort=25 velocity=37; origin xyz=0 -0.04 0 rpy=0 0 0 -> xyz=0 -0.038 -0.013831 rpy=0.27925 0 0
- joint right_shoulder_yaw_joint: limit lower=-2.62 upper=2.62 effort=40 velocity=32 -> lower=-2.618 upper=2.618 effort=25 velocity=37; origin xyz=0 0 0 rpy=0 0 0 -> xyz=0 -0.00624 -0.1032 rpy=0 0 0
- joint right_wrist_roll_joint: axis 0 0 1 -> 1 0 0; child right_wrist_roll_link -> right_wrist_roll_rubber_hand; limit lower=-1.97 upper=1.97 effort=18 velocity=32 -> lower=-1.972222054 upper=1.972222054 effort=25 velocity=37; origin xyz=0 0 -0.18 rpy=0 0 0 -> xyz=0.100 -0.00188791 -0.010 rpy=0 0 0
- joint waist_yaw_joint: limit lower=-2.62 upper=2.62 effort=88 velocity=32 -> lower=-2.618 upper=2.618 effort=88 velocity=32; origin xyz=0 0 0.06 rpy=0 0 0 -> xyz=-0.0039635 0 0.054 rpy=0 0 0

File: examples/unitree-go2.urdf (robot description, URDF)
Before this commit: robot unitree_go2, 17 links, 16 joints
Links:
- removed link trunk
- added link FL_calf_rotor, mass 0.089
- added link FL_calflower; collision cylinder length=0.065 radius=0.011
- added link FL_calflower1; collision cylinder length=0.03 radius=0.0155
- added link FL_hip_rotor, mass 0.089
- added link FL_thigh_rotor, mass 0.089
- added link FR_calf_rotor, mass 0.089
- added link FR_calflower; collision cylinder length=0.065 radius=0.011
- added link FR_calflower1; collision cylinder length=0.03 radius=0.0155
- added link FR_hip_rotor, mass 0.089
- added link FR_thigh_rotor, mass 0.089
- added link Head_lower, mass 0.001; collision sphere radius=0.047
- added link Head_upper, mass 0.001; collision cylinder length=0.09 radius=0.05
- added link RL_calf_rotor, mass 0.089
- added link RL_calflower; collision cylinder length=0.065 radius=0.011
- added link RL_calflower1; collision cylinder length=0.03 radius=0.0155
- added link RL_hip_rotor, mass 0.089
- added link RL_thigh_rotor, mass 0.089
- added link RR_calf_rotor, mass 0.089
- added link RR_calflower; collision cylinder length=0.065 radius=0.011
- added link RR_calflower1; collision cylinder length=0.03 radius=0.0155
- added link RR_hip_rotor, mass 0.089
- added link RR_thigh_rotor, mass 0.089
- added link base, mass 6.921; collision box size=0.3762 0.0935 0.114; visual mesh filename=package://go2_description/dae/base.dae
- added link front_camera
- added link imu, mass 0
- added link radar, mass 0
- link FL_calf: mass 0.16 -> 0.154; geometry collision cylinder length=0.12 radius=0.012; visual mesh filename=package://go2_description/dae/calf.dae
- link FL_foot: mass 0.06 -> 0.04; geometry collision sphere radius=0.022; visual mesh filename=package://go2_description/dae/foot.dae
- link FL_hip: mass 0.68 -> 0.678; geometry collision cylinder length=0.04 radius=0.046; visual mesh filename=package://go2_description/dae/hip.dae
- link FL_thigh: mass 1.15 -> 1.152; geometry collision box size=0.213 0.0245 0.034; visual mesh filename=package://go2_description/dae/thigh.dae
- link FR_calf: mass 0.16 -> 0.154; geometry collision cylinder length=0.12 radius=0.013; visual mesh filename=package://go2_description/dae/calf_mirror.dae
- link FR_foot: mass 0.06 -> 0.04; geometry collision sphere radius=0.022; visual mesh filename=package://go2_description/dae/foot.dae
- link FR_hip: mass 0.68 -> 0.678; geometry collision cylinder length=0.04 radius=0.046; visual mesh filename=package://go2_description/dae/hip.dae
- link FR_thigh: mass 1.15 -> 1.152; geometry collision box size=0.213 0.0245 0.034; visual mesh filename=package://go2_description/dae/thigh_mirror.dae
- link RL_calf: mass 0.16 -> 0.154; geometry collision cylinder length=0.12 radius=0.013; visual mesh filename=package://go2_description/dae/calf.dae
- link RL_foot: mass 0.06 -> 0.04; geometry collision sphere radius=0.022; visual mesh filename=package://go2_description/dae/foot.dae
- link RL_hip: mass 0.68 -> 0.678; geometry collision cylinder length=0.04 radius=0.046; visual mesh filename=package://go2_description/dae/hip.dae
- link RL_thigh: mass 1.15 -> 1.152; geometry collision box size=0.213 0.0245 0.034; visual mesh filename=package://go2_description/dae/thigh.dae
- link RR_calf: mass 0.16 -> 0.154; geometry collision cylinder length=0.12 radius=0.013; visual mesh filename=package://go2_description/dae/calf_mirror.dae
- link RR_foot: mass 0.06 -> 0.04; geometry collision sphere radius=0.022; visual mesh filename=package://go2_description/dae/foot.dae
- link RR_hip: mass 0.68 -> 0.678; geometry collision cylinder length=0.04 radius=0.046; visual mesh filename=package://go2_description/dae/hip.dae
- link RR_thigh: mass 1.15 -> 1.152; geometry collision box size=0.213 0.0245 0.034; visual mesh filename=package://go2_description/dae/thigh_mirror.dae
Joints:
- removed joint FL_foot_fixed_joint
- removed joint FR_foot_fixed_joint
- removed joint RL_foot_fixed_joint
- removed joint RR_foot_fixed_joint
- added joint FL_calf_rotor_joint: type fixed, parent FL_thigh, child FL_calf_rotor, origin xyz=0 -0.03235 0 rpy=0 0 0
- added joint FL_calflower1_joint: type fixed, parent FL_calflower, child FL_calflower1, origin xyz=-0.01 0 -0.04 rpy=0 0.48 0, axis 0 0 0
- added joint FL_calflower_joint: type fixed, parent FL_calf, child FL_calflower, origin xyz=0.020 0 -0.148 rpy=0 0.05 0, axis 0 0 0
- added joint FL_foot_joint: type fixed, parent FL_calf, child FL_foot, origin xyz=0 0 -0.213 rpy=0 0 0, axis 0 0 0
- added joint FL_hip_rotor_joint: type fixed, parent base, child FL_hip_rotor, origin xyz=0.11215 0.04675 0 rpy=0 0 0
- added joint FL_thigh_rotor_joint: type fixed, parent FL_hip, child FL_thigh_rotor, origin xyz=0 -0.00015 0 rpy=0 0 0
- added joint FR_calf_rotor_joint: type fixed, parent FR_thigh, child FR_calf_rotor, origin xyz=0 0.03235 0 rpy=0 0 0
- added joint FR_calflower1_joint: type fixed, parent FR_calflower, child FR_calflower1, origin xyz=-0.01 0 -0.04 rpy=0 0.48 0, axis 0 0 0
- added joint FR_calflower_joint: type fixed, parent FR_calf, child FR_calflower, origin xyz=0.020 0 -0.148 rpy=0 0.05 0, axis 0 0 0
- added joint FR_foot_joint: type fixed, parent FR_calf, child FR_foot, origin xyz=0 0 -0.213 rpy=0 0 0, axis 0 0 0
- added joint FR_hip_rotor_joint: type fixed, parent base, child FR_hip_rotor, origin xyz=0.11215 -0.04675 0 rpy=0 0 0
- added joint FR_thigh_rotor_joint: type fixed, parent FR_hip, child FR_thigh_rotor, origin xyz=0 0.00015 0 rpy=0 0 0
- added joint Head_lower_joint: type fixed, parent Head_upper, child Head_lower, origin xyz=0.008 0 -0.07 rpy=0 0 0, axis 0 0 0
- added joint Head_upper_joint: type fixed, parent base, child Head_upper, origin xyz=0.285 0 0.01 rpy=0 0 0, axis 0 0 0
- added joint RL_calf_rotor_joint: type fixed, parent RL_thigh, child RL_calf_rotor, origin xyz=0 -0.03235 0 rpy=0 0 0
- added joint RL_calflower1_joint: type fixed, parent RL_calflower, child RL_calflower1, origin xyz=-0.01 0 -0.04 rpy=0 0.48 0, axis 0 0 0
- added joint RL_calflower_joint: type fixed, parent RL_calf, child RL_calflower, origin xyz=0.020 0 -0.148 rpy=0 0.05 0, axis 0 0 0
- added joint RL_foot_joint: type fixed, parent RL_calf, child RL_foot, origin xyz=0 0 -0.213 rpy=0 0 0, axis 0 0 0
- added joint RL_hip_rotor_joint: type fixed, parent base, child RL_hip_rotor, origin xyz=-0.11215 0.04675 0 rpy=0 0 0
- added joint RL_thigh_rotor_joint: type fixed, parent RL_hip, child RL_thigh_rotor, origin xyz=0 -0.00015 0 rpy=0 0 0
- added joint RR_calf_rotor_joint: type fixed, parent RR_thigh, child RR_calf_rotor, origin xyz=0 0.03235 0 rpy=0 0 0
- added joint RR_calflower1_joint: type fixed, parent RR_calflower, child RR_calflower1, origin xyz=-0.01 0 -0.04 rpy=0 0.48 0, axis 0 0 0
- added joint RR_calflower_joint: type fixed, parent RR_calf, child RR_calflower, origin xyz=0.020 0 -0.148 rpy=0 0.05 0, axis 0 0 0
- added joint RR_foot_joint: type fixed, parent RR_calf, child RR_foot, origin xyz=0 0 -0.213 rpy=0 0 0, axis 0 0 0
- added joint RR_hip_rotor_joint: type fixed, parent base, child RR_hip_rotor, origin xyz=-0.11215 -0.04675 0 rpy=0 0 0
- added joint RR_thigh_rotor_joint: type fixed, parent RR_hip, child RR_thigh_rotor, origin xyz=0 0.00015 0 rpy=0 0 0
- added joint front_camera_joint: type fixed, parent base, child front_camera, origin xyz=0.32715 -0.00003 0.04297 rpy=0 0 0
- added joint imu_joint: type fixed, parent base, child imu, origin xyz=-0.02557 0 0.04232 rpy=0 0 0, axis 0 0 0
- added joint radar_joint: type fixed, parent base, child radar, origin xyz=0.28945 0 -0.046825 rpy=0 2.8782 0, axis 0 0 0
- joint FL_calf_joint: limit lower=-2.7227 upper=-0.83776 effort=35.55 velocity=20.07 -> lower=-2.7227 upper=-0.83776 effort=45.43 velocity=15.70
- joint FL_hip_joint: parent trunk -> base
- joint FR_calf_joint: limit lower=-2.7227 upper=-0.83776 effort=35.55 velocity=20.07 -> lower=-2.7227 upper=-0.83776 effort=45.43 velocity=15.70
- joint FR_hip_joint: parent trunk -> base
- joint RL_calf_joint: limit lower=-2.7227 upper=-0.83776 effort=35.55 velocity=20.07 -> lower=-2.7227 upper=-0.83776 effort=45.43 velocity=15.70
- joint RL_hip_joint: parent trunk -> base
- joint RR_calf_joint: limit lower=-2.7227 upper=-0.83776 effort=35.55 velocity=20.07 -> lower=-2.7227 upper=-0.83776 effort=45.43 velocity=15.70
- joint RR_hip_joint: parent trunk -> base
